File: PDR-voltage tranmitter/Voltage Transmitter-schematic.sch (KiCad schematic (older format))
At the start: 5 parts

Commit message: hopefully last commit before PDR
Parts:
- added Conn?: Battery Pack, symbol Voltage-Transmitter-schematic-rescue:Molex_SL_02-MRDT_Connectors
- added R1: 40k, symbol Device:R_Small
- added R2: 7k, symbol Device:R_Small
- Conn?: symbol MRDT_Connectors:Molex_SL_02 -> Voltage-Transmitter-schematic-rescue:Molex_SL_02-MRDT_Connectors
- U?: symbol MRDT_Shields:Raspberry_Pi -> Voltage-Transmitter-schematic-rescue:Raspberry_Pi-MRDT_Shields
- U?: symbol MRDT_ICs:AP1059 -> Voltage-Transmitter-schematic-rescue:AP1059-MRDT_ICs
Connections:
- net GND: now also U?.3 (FB), U?.4 (SD), Conn?.1, R2.2; no longer U?.14 (GND), U?.20 (GND), U?.25 (GND), U?.30 (GND), U?.34 (GND), U?.39 (GND), U?.6 (GND)
- net VBATT: now reaches C1.2, Conn?.1, U?.1 (Vin)
- net VOUT renamed V_Sense
- net V_Sense: now also R1.1, R2.1
- new net PV_In: Conn?.2, R1.2
Other:
- note added: "2 LiPo Batteries\n"
- note added: "Voltage Divider\n"
- note added: "Voltage Regulator\n"
- moved on the sheet: C1, Conn?, U?
