File: voltage tranmitter/Voltage Transmitter-schematic.sch (KiCad schematic (older format))
At the start: 11 parts, among them U1 AP1059, U2 ESP8266_MCU

Commit message: Changes since First Board Review
Parts:
- U2: footprint New Library:ESP_8266 NODEMCU -> VoltageTransmitter_Hardware:ESP_8266 NODEMCU
Changed lines of the file:
@@
 F 0 "U2" H 3975 1325 50  0000 C CNN
 F 1 "ESP8266_MCU" H 3975 1234 50  0000 C CNN
-F 2 "New Library:ESP_8266 NODEMCU" H 3700 1300 50  0001 C CNN
+F 2 "VoltageTransmitter_Hardware:ESP_8266 NODEMCU" H 3700 1300 50  0001 C CNN
 F 3 "" H 3700 1300 50  0001 C CNN
 	1    3700 1300
