File: voltage tranmitter/VoltageTransmitter_Hardware.kicad_pcb (KiCad board)
At the start: 2 copper layers, 11 parts, among them U1 AP1059, U2 ESP8266_MCU

Commit message: Change the footprint on the ESP8266-added silkscreen
Parts:
- Conn1: value AndersonPP -> AndersonPP-MRDT_Connectors
Connections:
- Conn1 pad 2: (no net) -> Net-(Conn1-Pad2)
- R1 pad 1: Net-(Conn3-Pad2) -> Net-(Conn1-Pad2)
Changed lines of the file:
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@@
   )
   (setup
-    (last_trace_width 0.762)
+    (last_trace_width 0.25)
     (user_trace_width 0.381)
     (user_trace_width 0.762)
@@
     (pad_drill 0.6)
     (pad_to_mask_clearance 0)
+    (solder_mask_min_width 0.25)
     (aux_axis_origin 0 0)
-    (visible_elements FFFFFF7F)
+    (visible_elements 7FFFFFFF)
     (pcbplotparams
       (layerselection 0x010fc_ffffffff)
@@
   (net 31 "Net-(U2-Pad29)")
   (net 32 "Net-(U2-Pad30)")
-  (net 33 "Net-(Conn3-Pad2)")
+  (net 33 "Net-(Conn1-Pad2)")
   (net_class Default "This is the default net class."
     (clearance 0.2)
@@
     (add_net GND)
     (add_net "Net-(C1-Pad1)")
-    (add_net "Net-(Conn3-Pad2)")
+    (add_net "Net-(Conn1-Pad2)")
     (add_net "Net-(D1-Pad1)")
     (add_net "Net-(U2-Pad1)")
@@
       (effects (font (size 1 1) (thickness 0.15)))
     )
-    (fp_text value AndersonPP (at -12.8651 -16.764 180) (layer F.Fab)
+    (fp_text value AndersonPP-MRDT_Connectors (at -12.8651 -16.764 180) (layer F.Fab)
       (effects (font (size 1 1) (thickness 0.15)))
     )
@@
     (pad 1 thru_hole circle (at 3.5814 -4.063 180) (size 5.08 5.08) (drill 4.06) (layers *.Cu *.Mask F.Paste)
       (net 2 GND))
-    (pad 2 thru_hole circle (at 3.5814 -12.064 180) (size 5.08 5.08) (drill 4.06) (layers *.Cu *.Mask F.Paste))
+    (pad 2 thru_hole circle (at 3.5814 -12.064 180) (size 5.08 5.08) (drill 4.06) (layers *.Cu *.Mask F.Paste)
+      (net 33 "Net-(Conn1-Pad2)"))
   )
   (module MRDT_Connectors:MOLEX_SL_02_Horizontal (layer F.Cu)
@@
     )
     (pad 1 smd roundrect (at -0.875 0 180) (size 1.05 0.95) (layers F.Cu F.Paste F.Mask) (roundrect_rratio 0.25)
-      (net 33 "Net-(Conn3-Pad2)"))
+      (net 33 "Net-(Conn1-Pad2)"))
     (pad 2 smd roundrect (at 0.875 0 180) (size 1.05 0.95) (layers F.Cu F.Paste F.Mask) (roundrect_rratio 0.25)
       (net 5 Din))

Commit message: yeet
Parts:
- U2: footprint New Library:ESP_8266 NODEMCU -> VoltageTransmitter_Hardware:ESP_8266 NODEMCU
- moved U2 49.4 mm to (126.4, 63.3)

Commit message: Did the traces for the PCB
Parts:
- removed Conn3: AndersonPP-MRDT_Connectors, MRDT_Connectors:Anderson_1_Horisontal
- removed D1: D_Schottky, Diode_SMD:D_0603_1608Metric_Pad1.05x0.95mm_HandSolder
- removed L1: 47uH, Inductor_SMD:L_0603_1608Metric_Pad1.05x0.95mm_HandSolder
- C1, C2, Conn1, Conn2, R1, R2: moved to B.Cu
- U1: value AP1059 -> OKI; footprint MRDT_Devices:AP1509 -> MRDT_Devices:OKI_Horizontal; moved to B.Cu
- moved Conn2 31.4 mm to (131.6, 104.6), turned to 0 degrees
- moved U1 29.9 mm to (122.9, 99.1)
- moved C1 24.4 mm to (126.0, 101.1)
- moved C2 19.7 mm to (129.9, 101.1)
- moved Conn1 18.9 mm to (140.2, 71.1), turned to 270 degrees
- moved U2 18.5 mm to (144.8, 61.0)
- moved R1 11.5 mm to (129.2, 79.8), turned to 0 degrees
- moved R2 5.33 mm to (135.3, 79.8)
Connections:
- C1 pad 2: GND -> Net-(C1-Pad2)
- C2 pad 1: GND -> +3V3
- C2 pad 2: +3V3 -> Net-(C1-Pad2)
- Conn2 pad 1: Net-(C1-Pad1) -> Net-(C1-Pad2)
- Conn2 pad 2: GND -> Net-(C1-Pad1)
- U1 pad 2: Net-(D1-Pad1) -> Net-(C1-Pad2)
- U2 pad 1: Net-(U2-Pad1) -> Din
- U2 pad 12: Din -> Net-(U2-Pad12)
- U2 pad 24: Net-(U2-Pad24) -> GND
Routing:
- net Din: track 8.38 -> 35.6 mm
- net +3V3: track 12.7 -> 34.3 mm
- net Net-(C1-Pad1): track 1.65 -> 17.8 mm
- net Net-(C1-Pad2): track 0.00 -> 9.96 mm
- net Net-(D1-Pad1): track 5.18 -> 0.00 mm
- net Net-(Conn1-Pad2): track 0.00 -> 5.12 mm
- net GND: track 0.00 -> 5.06 mm
Other:
- board outline added: 30.5 x 61 mm
