File: Voltage Transmitter/VoltageTransmitter_Hardware.sch (KiCad schematic (older format))
At the start: 8 parts, among them U1 OKI, U2 ESP8266_MCU

Commit message: Gerbs Made
Connections:
- net labels removed: PV_In, V_Sense
Other:
- note added: "+8.2 V in"
Changed lines of the file:
@@
 Text Notes 500  650  0    118  ~ 24
 Voltage Regulator\n
-Text Label 2250 2600 2    50   ~ 0
-V_Sense
-Text Label 1950 2700 0    50   ~ 0
-PV_In
 $Comp
 L VoltageTransmitter_Hardware-rescue:ESP8266_MCU-New_libraries-Voltage-Transmitter-schematic-rescue-Voltage-Transmitter-schematic-rescue U2
@@
 	1650 2600 1700 2600
 Wire Wire Line
-	1900 2600 1950 2600
-Wire Wire Line
 	1950 2700 1950 2600
 $Comp
@@
 	1    0    0    -1
 $EndComp
-Connection ~ 1950 2600
 Wire Wire Line
 	1650 3000 1950 3000
@@
 Text GLabel 2300 2600 2    50   Output ~ 0
 Din
-Wire Wire Line
-	1950 2600 2300 2600
 $Comp
 L power:GND #PWR0104
@@
 	2650 1150 2650 1200
 Connection ~ 2650 1200
+Connection ~ 1950 2600
+Wire Wire Line
+	1950 2600 2300 2600
+Wire Wire Line
+	1900 2600 1950 2600
+Text Notes 850  1550 0    50   ~ 0
++8.2 V in
+$Comp
+L power:GND #PWR0106
+U 1 1 5C1A8175
+P 2150 1500
+F 0 "#PWR0106" H 2150 1250 50  0001 C CNN
+F 1 "GND" H 2155 1327 50  0000 C CNN
+F 2 "" H 2150 1500 50  0001 C CNN
+F 3 "" H 2150 1500 50  0001 C CNN
+	1    2150 1500
+	1    0    0    -1
+$EndComp
 $EndSCHEMATC

Commit message: Changed shaped & added comps
Changed to stacked andersons, added power led, transmitting led, and made sure no comps are located on the bottom of the board.
Parts:
- added D1, D2: LED, LED_SMD:LED_0603_1608Metric_Pad1.05x0.95mm_HandSolder, symbol Device:LED
- added R3, R4: 500, Resistor_SMD:R_0603_1608Metric_Pad1.05x0.95mm_HandSolder, symbol Device:R_Small
- added SW1: SW_Push_SPDT, Button_Switch_THT:SW_CuK_OS102011MA1QN1_SPDT_Angled, symbol Switch:SW_Push_SPDT
- Conn1: footprint MRDT_Connectors:Anderson_2_Horisontal_Side_by_Side -> MRDT_Connectors:Anderson_2_Horizontal_Stacked
- R1: value 100K -> 150K
- R2: value 11K -> 15K
Connections:
- net labels added: TX_IND
- wire segments 20 -> 30
- no-connect marks 0 -> 25
Other:
- note added: "9V Battery\n"
- note added: "Blue"
- note added: "ESP8266-12e\n"
- note added: "Green"
- note added: "Indication\n"
- note added: "Power Input\n\n"
- note added: "Switched andersons so that \nthey properly mate with the \nandersons on the batt packs"
- note added: "Voltage Sensing\n"
- note removed: "+8.2 V in"
- note removed: "2 LiPo Batteries\n"
- note removed: "ESP8266\n"
- note removed: "Voltage Divider\n"
- note removed: "Voltage Regulator\n"
- moved on the sheet: Conn1A, Conn1B, Conn2, U2
